Commit message: Update gmapbot.xacro

File: urdf/gmapbot.xacro (robot description, xacro)
@@ -192,5 +192,5 @@
       <origin xyz="0 0 0" rpy="0 0 0"/>
       <geometry>
-        <mesh filename="package://chapter7_tutorials/meshes/hokuyo.dae"/>
+        <mesh filename="package://gslambot/meshes/hokuyo.dae"/>
       </geometry>
     </visual>
